File: galvoDriver/galvoDriver.kicad_pcb (KiCad board)
At the start: 2 copper layers, 26 parts, among them U1 LM358, U2 LM358, U3 LM358

Commit message: Updated placement
Parts:
- moved JP5 38.2 mm to (170.2, 86.4)
- moved JP4 32.6 mm to (170.2, 101.6)
- moved C2 29.2 mm to (143.5, 86.4), turned to 90 degrees
- moved R12 28.5 mm to (165.1, 83.8)
- moved R8 26.6 mm to (165.1, 88.9), turned to 90 degrees
- moved R2 25.3 mm to (143.5, 81.3), turned to 270 degrees
- moved R5 25.3 mm to (160.0, 99.1), turned to 270 degrees
- moved R7 24.5 mm to (160.0, 83.8), turned to 270 degrees
- moved U3 24.2 mm to (149.9, 83.8), turned to 270 degrees
- moved R4 24.0 mm to (160.0, 88.9)
- moved R3 23.8 mm to (160.0, 104.1)
- moved RV2 22.7 mm to (138.4, 83.8), turned to 0 degrees
- moved R11 21.2 mm to (165.1, 99.1)
- moved JP3 21.1 mm to (132.1, 83.8)
- moved RV4 21.1 mm to (152.4, 91.4), turned to 90 degrees
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Connections:
- U1 pad 1: Net-(R1-Pad2) -> Net-(R2-Pad2)
- U1 pad 2: Net-(RV1-Pad2) -> Net-(RV2-Pad2)
- U1 pad 3: /xin -> /yin
- U1 pad 5: /yin -> /xin
- U1 pad 6: Net-(RV2-Pad2) -> Net-(RV1-Pad2)
- U1 pad 7: Net-(R2-Pad2) -> Net-(R1-Pad2)

Commit message: First pass at layout finished
Parts:
- moved C1 2.40 mm to (141.2, 106.0), turned to 270 degrees
- moved JP2 2.40 mm to (129.8, 93.3)
- moved R11 2.40 mm to (162.8, 98.4)
- moved R4 2.40 mm to (157.7, 88.2)
- moved R5 2.40 mm to (157.7, 98.4)
- moved R8 2.40 mm to (162.8, 88.2)
- moved R9 2.40 mm to (152.6, 98.4)
- moved RV3 2.40 mm to (150.1, 106.0)
- moved U2 2.40 mm to (147.6, 98.4)
- moved C2 2.40 mm to (141.2, 85.7)
- moved JP1 2.40 mm to (129.8, 103.5)
- moved JP3 2.40 mm to (129.8, 83.2)
- moved JP4 2.40 mm to (167.9, 100.9)
- moved JP5 2.40 mm to (167.9, 85.7)
- moved R1 2.40 mm to (141.2, 100.9)
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Routing:
- net VCC: track 0.00 -> 53.4 mm, vias 0 -> 2
- net Net-(R12-Pad2): track 0.00 -> 25.4 mm
- net /xout-: track 0.00 -> 24.2 mm
- net Net-(R11-Pad2): track 0.00 -> 23.8 mm
- net /yout-: track 0.00 -> 23.8 mm
- net /yout+: track 0.00 -> 21.3 mm
- net /xout+: track 0.00 -> 21.3 mm
- net GND: track 0.00 -> 16.4 mm, vias 0 -> 10
- net Net-(R4-Pad1): track 0.00 -> 15.3 mm
- net Net-(R3-Pad1): track 0.00 -> 15.0 mm
- net Net-(R1-Pad1): track 0.00 -> 14.0 mm
- net Net-(R10-Pad2): track 0.00 -> 13.8 mm
- net Net-(R1-Pad2): track 0.00 -> 13.5 mm
- net Net-(R2-Pad2): track 0.00 -> 12.2 mm
- net Net-(C1-Pad1): track 0.00 -> 12.2 mm
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- added copper zone on B.Cu, net GND
Other:
- board outline added: 43.8 x 31.1 mm
- net class Default: clearance 0.2 -> 0.1778; trace_width 0.25 -> 0.1524; via_dia 0.6 -> 0.381; via_drill 0.4 -> 0.3302
- rule trace_clearance: 0.2 -> 0.1778
- rule trace_min: 0.2 -> 0.1524
- rule via_min_drill: 0.3 -> 0.3302
- rule via_min_size: 0.4 -> 0.381
- board text added: "GND"
- board text added: "V+"
- board text added: "X+"
- board text added: "X-"
- board text added: "Xin"
- board text added: "Y+"
- board text added: "Y-"
- board text added: "Yin"

Commit message: Added rear silkscreen
Other:
- board text added: "defconbots galvo controller v2.0 by @alvaroprieto alvarop.com"
Changed lines of the file:
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@@
   (general
     (links 54)
-    (no_connects 12)
+    (no_connects 0)
     (area 126.949999 78.054999 170.865001 109.270001)
     (thickness 1.6)
-    (drawings 12)
+    (drawings 13)
     (tracks 195)
     (zones 0)
@@
     (visible_elements FFFFFF7F)
     (pcbplotparams
-      (layerselection 0x00030_80000001)
-      (usegerberextensions false)
+      (layerselection 0x010fc_80000001)
+      (usegerberextensions true)
       (excludeedgelayer true)
       (linewidth 0.100000)
@@
       (outputformat 1)
       (mirror false)
-      (drillshape 1)
+      (drillshape 0)
       (scaleselection 1)
-      (outputdirectory ""))
+      (outputdirectory grb/))
   )
   (net 0 "")
@@
     )
   )
+  (gr_text "defconbots galvo controller v2.0\nby @alvaroprieto\nalvarop.com\n" (at 149.86 83.82) (layer B.SilkS)
+    (effects (font (size 1.5 1.5) (thickness 0.3)) (justify mirror))
+  )
   (gr_text GND (at 130 98.5) (layer F.SilkS)
